File: 1.Hardware/MSP432.kicad_sch (KiCad schematic)
At the start: 39 parts, among them IC1 SN74LVC244APW, J1 PWR, J2 MOTOR, SW1 SW_DPDT, SW3 SW_5DIR, U1 AMS1117-3.3, U2 LM1085-ADJ, U3 LM2940S-5.0, U4 MSP-EXP432P401R

Commit message: grand upgrade of both firmware and hardware
Parts:
- removed C1, C10, C2, C6: 10uF, symbol Device:C_Polarized_Small_US
- removed C12, C3, C4, C8: 0.1uF, symbol Device:C_Small
- removed C13, C5, C9: 22uF, symbol Device:C_Polarized_Small_US
- removed C14: 470uF, symbol Device:C_Polarized_Small_US
- removed D1, D2: LED, symbol Device:LED
- removed D3: 1N4148, Diode_SMD:D_SMA, symbol Simulation_SPICE:DIODE
- removed IC1: SN74LVC244APW, symbol ErBW_s:SN74LVC244APW
- removed J1: PWR, Connector:VCC_CONN, symbol Connector_Generic:Conn_01x02
- removed J2: MOTOR, Connector:VCC_CONN, symbol Connector_Generic:Conn_01x02
- removed J?: TFT, Connector_PinSocket_2.54mm:PinSocket_1x08_P2.54mm_Vertical, symbol ErBW_s:Display_Socket_1x8_2.54mm
- removed R1, R5: 5K1, symbol Device:R_Small
- removed R3: 1K, symbol Device:R_Small
- removed R4: 0R, Resistor_SMD:R_1206_3216Metric_Pad1.30x1.75mm_HandSolder, symbol Device:R_Small
- removed RV1: 3296W, symbol Device:R_Potentiometer
- removed SW1: SW_DPDT, symbol Switch:SW_DPDT_x2
- removed SW3: SW_5DIR, Button_Switch_SMD:SW_5DIR, symbol Switch:SW_5DIR
- removed TP1: 6V, TestPoint:TestPoint_Pad_D2.5mm, symbol Connector:TestPoint
- removed TP2: 5V, TestPoint:TestPoint_Pad_D2.5mm, symbol Connector:TestPoint
- removed TP3: 3V3, TestPoint:TestPoint_Pad_D2.5mm, symbol Connector:TestPoint
- removed TP4: GND, TestPoint:TestPoint_Pad_2.5x2.5mm, symbol Connector:TestPoint
- removed U1: AMS1117-3.3, symbol Regulator_Linear:AMS1117-3.3
- removed U2: LM1085-ADJ, symbol Regulator_Linear:LM1085-ADJ
- removed U3: LM2940S-5.0, symbol Regulator_Linear:LM2940S-5.0
- removed U4: MSP-EXP432P401R, Connector_PinHeader_2.54mm:MSP-EXP432P401R, symbol MCU_Texas_SimpleLink:MSP-EXP432P401R
- added C10: 10uF, Capacitor_SMD:C_0603_1608Metric, symbol Device:C_Small
- added C9: 100nF, Capacitor_SMD:C_0603_1608Metric, symbol Device:C_Small
- added D1: 1N4148W, Diode_SMD:D_SMA, symbol Diode:1N4148W
- added F?: 500mA, Fuse:Fuse_0603_1608Metric, symbol Device:Fuse_Small
- added J2, J6: Conn_01x06, Connector_PinHeader_2.54mm:PinHeader_1x06_P2.54mm_Vertical, symbol Connector_Generic:Conn_01x06
- added J3, J7: Conn_01x04, Connector_PinHeader_2.54mm:PinHeader_1x04_P2.54mm_Vertical, symbol Connector_Generic:Conn_01x04
- added J4: Conn_01x08, Connector_PinSocket_2.54mm:PinSocket_1x08_P2.54mm_Vertical, symbol Connector_Generic:Conn_01x08
- added J5: Conn_01x04, Connector_PinSocket_2.54mm:PinSocket_1x04_P2.54mm_Vertical, symbol Connector_Generic:Conn_01x04
- added J9: SERVO, Connector_PinHeader_2.54mm:PinHeader_1x03_P2.54mm_Vertical, symbol Connector_Generic:Conn_01x03
- added Q1: S8050, Package_TO_SOT_SMD:SOT-23, symbol Transistor_BJT:2N3055
- added R11, R21: 5K1, Resistor_SMD:R_0603_1608Metric, symbol Device:R_Small
- added R6: 1K, Resistor_SMD:R_0603_1608Metric, symbol Device:R_Small
- added SW1: SW_SPDT, ErBW_s:SPDT_MTS_102, symbol Switch:SW_SPDT
- added SW2, SW3, SW4: 3x4, ErBW_s:BUTTON_3x4, symbol Switch:SW_Push
- added U2: RT9013-33GB, Package_TO_SOT_SMD:SOT-23-5, symbol ErBW_s:RT9013-33GB
- added U2: MSP-EXP432P401R, ErBW_s:MSP-EXP432P401R, symbol ErBW_s:MSP-EXP432P401R
- BZ1: footprint Buzzer_Beeper:Buzzer_9*9P5 -> ErBW_s:DET-402-G-1
- C11: value 0.1uF -> 10nF; footprint (none) -> Capacitor_SMD:C_0603_1608Metric
- C7: value 0.1uF -> 10uF; footprint (none) -> Capacitor_SMD:C_0603_1608Metric
- D4: footprint (none) -> LED_SMD:LED_0603_1608Metric
- R2: value 5K1 -> 10K; footprint (none) -> Resistor_SMD:R_0603_1608Metric
Connections:
- net +6V is gone; now on net +5V: R2.1
- net +3V3: now also BZ1.1 (-), C10.1, C9.1, R11.1, U2.5 (VOUT)
- net +5V: now also D1.1 (K), J3.4 (Pin_4), J4.2 (Pin_2), J5.4 (Pin_4), J6.1 (Pin_1), J7.1 (Pin_1), J9.2 (Pin_2), U2.1 (VIN), U2.3 (EN), U2.73 (5V), U2.74 (5V); no longer C7.1
- net GND: now also C11.2, C7.1, D4.1 (K), C10.2, C9.2, J2.3 (Pin_3), J2.4 (Pin_4), J3.3 (Pin_3), J4.1 (Pin_1), J5.3 (Pin_3), J6.2 (Pin_2), J7.2 (Pin_2), J9.1 (Pin_1), Q1.2 (E), R21.2, R6.2, SW2.2, SW3.2, SW4.2, U2.2 (GND), U2.20 (GND), U2.22 (GND), U2.77 (GND), U2.78 (GND)
- net VBUS: now also SW1.2 (B)
- net at D4.2 (A): now also R11.2
- net at BZ1.2 (+): now also Q1.3 (C)
- net BATTERY: now reaches R2.2
- net BATTERY: now also C7.2, R6.1, U2.49 (P5.3/A2)
- removed net GNDPWR: C11.2, C7.2, D4.1 (K)
- net VCC: no longer names the net of C11.1
- net VCC: now also U2.4 (NC)
- new net: D1.2 (A), SW1.1 (A)
- new net: F?.2, J9.3 (Pin_3)
- new net A2_RX: J5.2 (Pin_2), U2.3 (P3.2/PM_UCA2RXD/PM_UCA2SOMI)
- new net A2_TX: J5.1 (Pin_1), U2.4 (P3.3/PM_UCA2TXD/PM_UCA2SIMO)
- new net A3_RX: J3.2 (Pin_2), U2.60 (P9.6/UCA3RXD/UCA3SOMI)
- new net A3_TX: J3.1 (Pin_1), U2.61 (P9.7/UCA3TXD/UCA3SIMO)
- new net AUX_SCL: J7.3 (Pin_3), U2.23 (P6.1/A14)
- new net AUX_SDA: J7.4 (Pin_4), U2.24 (P4.0/A13)
- new net BUZZER: Q1.1 (B), R21.1, U2.17 (P5.7/TA2.2/VREF-/VEREF-/C1.6)
- new net DIR1: J2.2 (Pin_2), U2.64 (P7.4/PM_TA1.4/C0.5)
- new net DIR2: J2.6 (Pin_6), U2.66 (P7.6/PM_TA1.2/C0.3)
- new net ENCODER_A: SW2.1, U2.46 (P8.4/A21)
- new net ENCODER_B: SW3.1, U2.42 (P8.5/A20)
- new net IMU_CS: J6.6 (Pin_6), U2.33 (P5.1/A4)
- new net IMU_SDI: J6.4 (Pin_4), U2.36 (P6.6/TA2.3/UCB3SIMO/UCB3SDA/C1.1)
- new net IMU_SDO: J6.5 (Pin_5), U2.35 (P6.7/TA2.4/UCB3SOMI/UCB3SCL/C1.0)
- new net IMU_SPC: J6.3 (Pin_3), U2.67 (P10.1/UCB3CLK)
- new net IPS_CS: J4.7 (Pin_7), U2.31 (P3.7/PM_UCB2SOMI/PM_UCB2SCL)
- new net IPS_DC: J4.6 (Pin_6), U2.13 (P5.0/A5)
- new net IPS_RES: J4.5 (Pin_5), U2.12 (P5.2/A3)
- new net IPS_SCL: J4.3 (Pin_3), U2.32 (P3.5/PM_UCB2CLK)
- new net IPS_SDA: J4.4 (Pin_4), U2.11 (P3.6/PM_UCB2SIMO/PM_UCB2SDA)
- new net KEY_CENTER: SW4.1, U2.44 (P9.0/A17)
- new net PWM1: J2.1 (Pin_1), U2.63 (P7.5/PM_TA1.3/C0.4)
- new net PWM2: J2.5 (Pin_5), U2.65 (P7.7/PM_TA1.1/C0.2)
- new net SERVO: F?.1, U2.51 (P9.3/TA3.4)
Other:
- note removed: "BUTTON"
- note removed: "ISOLATION"
- note removed: "PORT"
- note removed: "REGULATOR"
